File: hardware/shaw.kicad_pcb (KiCad board)
At the start: 2 copper layers, 46 parts, among them J1 USB_C_Receptacle_USB2.0_14P, J2 Conn_01x20, J3 Conn_01x20, J4 Conn_01x03, J5 Conn_01x02, SW1 SW_Push, U1 RP2040, U2 MCP1700x-330xxTT, U3 W25Q16JVSS, U4 BQ24074RGT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

Commit message: .
Parts:
- moved R6 120.8 mm to (130.6, 97.6)
- moved R1 120.6 mm to (137.0, 79.0), turned to -90 degrees
- moved R9 119.5 mm to (136.0, 91.2), turned to 180 degrees
- moved R7 119.1 mm to (130.6, 96.4)
- moved R11 118.7 mm to (136.0, 89.2), turned to 180 degrees
- moved R2 117.2 mm to (134.2, 79.0), turned to -90 degrees
- moved R8 117.2 mm to (131.2, 93.4), turned to -90 degrees
- moved J5 115.6 mm to (139.9, 87.0), turned to 90 degrees
- moved C18 113.7 mm to (133.2, 87.0), turned to -90 degrees
- moved R10 113.3 mm to (132.0, 87.0), turned to -90 degrees
- moved R12 112.3 mm to (131.0, 87.0), turned to -90 degrees
- moved R13 111.0 mm to (130.0, 88.0), turned to 90 degrees
- moved SW1 110.0 mm to (140.0, 93.0), turned to -90 degrees
- moved U4 106.1 mm to (132.4, 90.2)
- moved D2 102.5 mm to (136.5, 92.5), turned to 90 degrees
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Connections:
- C19 pad 1: Net-(C19-Pad1) -> Net-(J5-Pin_2)
- C19 pad 2: Net-(J5-Pin_2) -> GND
- U4 pad 2: Net-(C19-Pad1) -> Net-(J5-Pin_2)
- U4 pad 3: Net-(C19-Pad1) -> Net-(J5-Pin_2)
Routing:
- net +3V3: track 22.8 -> 109.7 mm, vias 1 -> 9
- net GPIO0: track 0.00 -> 37.6 mm
- net GPIO29_ADC3: track 0.00 -> 35.7 mm
- net GPIO1: track 0.00 -> 35.6 mm
- net BQ_OUT: track 0.00 -> 34.0 mm, vias 0 -> 2
- net VBUS: track 0.00 -> 33.8 mm
- net GPIO28_ADC2: track 0.00 -> 31.1 mm
- net GPIO2: track 0.00 -> 31.0 mm
- net GPIO3: track 0.00 -> 28.9 mm
- net GPIO4: track 0.00 -> 26.9 mm
- net GPIO27_ADC1: track 0.00 -> 26.5 mm
- net GPIO5: track 0.00 -> 25.4 mm
- net GPIO26_ADC0: track 0.00 -> 24.5 mm
- net GPIO6: track 0.00 -> 20.4 mm, vias 0 -> 1
- net GPIO8: track 0.00 -> 20.3 mm, vias 0 -> 1
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- added copper zone on B.Cu, net GND
- added copper zone on F.Cu, net GND

Commit message: .
Parts:
- moved C12 0.53 mm to (135.9, 99.9)
- moved D2 0.15 mm to (136.6, 92.6)
Routing:
- net +3V3: track 109.7 -> 110.9 mm, vias 9 -> 10
- net USB_D+: track 30.5 -> 29.5 mm
- net USB_D-: track 30.5 -> 29.5 mm
- net +1V1: track 24.4 -> 25.2 mm
- net GND: track 20.6 -> 20.2 mm, vias 20 -> 23
Other:
- board outline added: 24.6 x 51 mm

Commit message: .
Parts:
- C20: footprint Capacitor_SMD:C_0201_0603Metric -> Capacitor_SMD:C_0603_1608Metric
- moved R11 2.42 mm to (135.0, 87.0), turned to -90 degrees
- moved C20 0.86 mm to (135.5, 89.5), turned to 90 degrees
- moved D2 0.38 mm to (136.6, 93.0)
- moved R9 0.34 mm to (136.0, 91.5)
Routing:
- net GND: track 20.2 -> 18.3 mm, vias 23 -> 26
- net BQ_OUT: track 34.0 -> 32.5 mm
- net Net-(U4-ILIM): track 1.76 -> 2.42 mm
