File: hardware/shaw.kicad_sch (KiCad schematic)
At the start: 46 parts, among them J1 USB_C_Receptacle_USB2.0_14P, J2 Conn_01x20, J3 Conn_01x20, J4 Conn_01x03, J5 Conn_01x02, SW1 SW_Push, U1 RP2040, U2 MCP1700x-330xxTT, U3 W25Q16JVSS, U4 BQ24074RGT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

Commit message: .
Connections:
- net GND: now also C19.2
- net at J5.2 (Pin_2): now also C19.1, U4.2 (BAT), U4.3 (BAT); no longer C19.2
Other:
- moved on the sheet: C19
Changed lines of the file:
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@@
 	)
 	(junction
+		(at 64.77 111.76)
+		(diameter 0)
+		(color 0 0 0 0)
+	)
+	(junction
 		(at 121.92 45.72)
 		(diameter 0)
@@
 	(wire
 		(pts
+			(xy 64.77 111.76) (xy 64.77 114.3)
+		)
+		(stroke
+			(width 0)
+			(type default)
+		)
+	)
+	(wire
+		(pts
 			(xy 118.11 83.82) (xy 119.38 83.82)
 		)
@@
 	(wire
 		(pts
-			(xy 59.69 115.57) (xy 62.23 115.57)
-		)
-		(stroke
-			(width 0)
-			(type default)
-		)
-	)
-	(wire
-		(pts
 			(xy 49.53 45.72) (xy 49.53 48.26)
 		)
@@
 	(wire
 		(pts
-			(xy 261.62 93.98) (xy 259.08 93.98)
+			(xy 72.39 114.3) (xy 74.93 114.3)
 		)
 		(stroke
@@
 	(wire
 		(pts
-			(xy 260.35 129.54) (xy 260.35 139.7)
+			(xy 261.62 93.98) (xy 259.08 93.98)
 		)
 		(stroke
@@
 	(wire
 		(pts
-			(xy 49.53 43.18) (xy 50.8 43.18)
+			(xy 260.35 129.54) (xy 260.35 139.7)
 		)
 		(stroke
@@
 	(wire
 		(pts
-			(xy 69.85 115.57) (xy 69.85 111.76)
+			(xy 49.53 43.18) (xy 50.8 43.18)
 		)
 		(stroke
@@
 	(wire
 		(pts
+			(xy 74.93 114.3) (xy 74.93 115.57)
+		)
+		(stroke
+			(width 0)
+			(type default)
+		)
+	)
+	(wire
+		(pts
 			(xy 224.79 129.54) (xy 224.79 139.7)
 		)
@@
 	(wire
 		(pts
+			(xy 59.69 115.57) (xy 59.69 111.76)
+		)
+		(stroke
+			(width 0)
+			(type default)
+		)
+	)
+	(wire
+		(pts
 			(xy 46.99 134.62) (xy 102.87 134.62)
 		)
@@
 	(wire
 		(pts
+			(xy 59.69 111.76) (xy 64.77 111.76)
+		)
+		(stroke
+			(width 0)
+			(type default)
+		)
+	)
+	(wire
+		(pts
+			(xy 64.77 111.76) (xy 82.55 111.76)
+		)
+		(stroke
+			(width 0)
+			(type default)
+		)
+	)
+	(wire
+		(pts
 			(xy 180.34 88.9) (xy 182.88 88.9)
 		)
@@
 	(wire
 		(pts
-			(xy 69.85 111.76) (xy 82.55 111.76)
-		)
-		(stroke
-			(width 0)
-			(type default)
-		)
-	)
-	(wire
-		(pts
 			(xy 223.52 121.92) (xy 226.06 121.92)
 		)
@@
 	)
 	(symbol
+		(lib_id "power:GND")
+		(at 74.93 115.57 0)
+		(unit 1)
+		(exclude_from_sim no)
+		(in_bom yes)
+		(on_board yes)
+		(dnp no)
+		(fields_autoplaced yes)
+		(property "Reference" "#PWR033"
+			(at 74.93 121.92 0)
+			(effects
+				(font
+					(size 1.27 1.27)
+				)
+				(hide yes)
+			)
+		)
+		(property "Value" "GND"
+			(at 74.93 120.65 0)
+			(effects
+				(font
+					(size 1.27 1.27)
+				)
+			)
+		)
+		(property "Footprint" ""
+			(at 74.93 115.57 0)
+			(effects
+				(font
+					(size 1.27 1.27)
+				)
+				(hide yes)
+			)
+		)
+		(property "Datasheet" ""
+			(at 74.93 115.57 0)
+			(effects
+				(font
+					(size 1.27 1.27)
+				)
+				(hide yes)
+			)
+		)
+		(property "Description" "Power symbol creates a global label with name \"GND\" , ground"
+			(at 74.93 115.57 0)
+			(effects
+				(font
+					(size 1.27 1.27)
+				)
+				(hide yes)
+			)
+		)
+		(pin "1"
+		)
+		(instances
+			(project ""
+				(path "/848203ef-ff6b-47cd-ae45-62b97bad7637"
+					(reference "#PWR033")
+					(unit 1)
+				)
+			)
+		)
+	)
+	(symbol
 		(lib_id "power:+1V1")
 		(at 149.86 64.77 0)
@@
 	(symbol
 		(lib_id "Device:C")
-		(at 66.04 115.57 90)
+		(at 68.58 114.3 90)
 		(unit 1)
 		(exclude_from_sim no)
@@
 		(dnp no)
 		(property "Reference" "C19"
-			(at 66.04 109.728 90)
+			(at 68.58 111.252 90)
 			(effects
 				(font
@@
 		)
 		(property "Value" "4.7uF"
-			(at 66.04 112.268 90)
+			(at 68.58 117.348 90)
 			(effects
 				(font
@@
 		)
 		(property "Footprint" "Capacitor_SMD:C_0603_1608Metric"
-			(at 69.85 114.6048 0)
+			(at 72.39 113.3348 0)
 			(effects
 				(font
@@
 		)
 		(property "Datasheet" "~"
-			(at 66.04 115.57 0)
+			(at 68.58 114.3 0)
 			(effects
 				(font
@@
 		)
 		(property "Description" "Unpolarized capacitor"
-			(at 66.04 115.57 0)
+			(at 68.58 114.3 0)
 			(effects
 				(font

Commit message: .
Parts:
- C20: footprint Capacitor_SMD:C_0201_0603Metric -> Capacitor_SMD:C_0603_1608Metric
Changed lines of the file:
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@@
 			)
 		)
-		(property "Footprint" "Capacitor_SMD:C_0201_0603Metric"
+		(property "Footprint" "Capacitor_SMD:C_0603_1608Metric"
 			(at 73.66 105.7148 0)
 			(effects
